Commit message: 6.4Gazebo中完成机器人的仿真

File: install/my_robo_description/share/my_robo_description/URDF/ano_robo.urdf.xacro (robot description, xacro)
@@ -10,4 +10,7 @@
     <xacro:include filename="$(find my_robo_description)/URDF/body_/wheel.urdf.xacro"/>
     <xacro:include filename="$(find my_robo_description)/URDF/body_/wheel_wangxianglun.urdf.xacro"/>
+    <!--插件-->
+    <xacro:include filename="$(find my_robo_description)/URDF/plugins/gazebo_control_plugin.xacro"/>
+    <xacro:include filename="$(find my_robo_description)/URDF/plugins/gazebo_sensor_plugin.xacro"/>
     <xacro:base_xacro length="0.12" radius="0.1"/>
     <!--传感器-->
@@ -19,3 +22,5 @@
     <xacro:wheel_wangxianglun_xacro wheel_wangxianglun_name="right_wangxianglun_name" xyz="0.08 0 -0.076"/>
     <xacro:wheel_wangxianglun_xacro wheel_wangxianglun_name="left_wangxianglun_name" xyz="-0.08 0 -0.076"/>
+    <xacro:gazebo_control_plugin />
+    <xacro:gazebo_sensor_plugin />
 </robot>

File: install/my_robo_description/share/my_robo_description/URDF/body_/wheel.urdf.xacro (robot description, xacro)
@@ -44,4 +44,11 @@
             <axis xyz="0 1 0"/>
         </joint>
+        <gazebo reference ="${wheel_name}_joint">
+            <mu1 value="20.0"/>
+            <mu2 value="20.0"/>
+            <kp value="1000000000.0"/>
+            <kd value="1.0"/>
+            <material>Gazebo/Green</material>
+        </gazebo>
     </xacro:macro>
 </robot>

File: install/my_robo_description/share/my_robo_description/URDF/body_/wheel_wangxianglun.urdf.xacro (robot description, xacro)
@@ -44,4 +44,11 @@
             <axis xyz="0 1 0"/>
         </joint>
+         <gazebo reference ="${wheel_wangxianglun_name}_joint">
+            <mu1 value="0.0"/>
+            <mu2 value="0.0"/>
+            <kp value="1000000000.0"/>
+            <kd value="1.0"/>
+            <material>Gazebo/Green</material>
+        </gazebo>
     </xacro:macro>
 </robot>

File: install/my_robo_description/share/my_robo_description/URDF/sensor/camera.urdf.xacro (robot description, xacro)
@@ -37,4 +37,10 @@
             <xacro:box_interial m="0.1" w="0.02" h="0.15" d="0.02"/>
         </link>
+        <link name="camera_opt_link"></link>
+        <joint name="camera_opt_joint" type="fixed">
+            <parent link="camera_link"/>
+            <child link="camera_opt_link"/>
+            <origin xyz="0 0 0" rpy="${-pi/2} 0.0 ${-pi/2}"/>
+        </joint>
         <!-- 机器人的关节 用于组合机器人的部件 -->
         <joint name="camera_joint" type="fixed">
